File: hw/plinkyblackfront/plinkyblackfront.kicad_pcb (KiCad board)
At the start: 2 copper layers, 121.9 x 128.3 mm, 83 parts, among them J1 Conn_02x08_Odd_Even, J2 Conn_02x08_Odd_Even, J3 Conn_02x08_Top_Bottom, J4 Conn_01x02, M1 MountingHole_3.2mm_M3, M2 MountingHole_3.2mm_M3, M3 MountingHole_3.2mm_M3, M4 MountingHole_3.2mm_M3

Commit message: add oss text to pcbs
Other:
- net class Default removed
- board text added: "opensource"
- board text added: "this PCB is based on the opensource version of plinky available at https://github.com/plinkysynth/plinky_public this is not an official kit and is not officially supported"
