File: hw/plinkyblackfront/plinkyblackfront_bigholes.kicad_pcb (KiCad board)
At the start: 2 copper layers, 121.9 x 128.3 mm, 83 parts, among them J1 Conn_02x08_Odd_Even, J2 Conn_02x08_Odd_Even, J3 Conn_02x08_Top_Bottom, J4 Conn_01x02, M1 MountingHole_3.2mm_M3, M2 MountingHole_3.2mm_M3, M3 MountingHole_3.2mm_M3, M4 MountingHole_3.2mm_M3

Commit message: production adjustments and convert testjig to kicad7
Connections:
- J1 pad 11: (no net) -> unconnected-(J1-Pin_11-Pad11)
Other:
- board text added: "JLCJLCJLCJLC"

Commit message: touch sensors redesigned in attemt to increase edges linearity
Routing:
- net Net-(J1-Pin_15): track 131.0 -> 119.4 mm
- net Net-(J1-Pin_13): track 133.3 -> 138.2 mm
- net T2: track 34.7 -> 30.8 mm
- net T11: track 56.2 -> 55.6 mm
