File: hw/v2/plinkyblack.kicad_pcb (KiCad board)
At the start: 4 copper layers, 121.9 x 109.2 mm, 267 parts, among them J1 AudioJack2_SwitchT, J10 AudioJack2_SwitchT, J11 AudioJack2_SwitchT, J12 Conn_02x08_Odd_Even, J13 Conn_02x08_Odd_Even, J14 AudioJack2_SwitchT, J15 AudioJack2_SwitchT, J16 AudioJack2_SwitchT, J17 AudioJack2_SwitchT, J18 USB_B_Micro, J19 SJ1-3523N, J2 AudioJack2_SwitchT, J20 oled0.91, J21 SJ1-3523N, J22 AudioJack2_SwitchT, J23 AudioJack2_SwitchT, J24 USB_B_Micro, J25 Conn_01x16_Female, J26 SJ1-3523N, J27 SJ1-3523N, J3 AudioJack2_SwitchT, J4 AudioJack2_SwitchT, J5 SWD header, J6 AudioJack2_SwitchT, J7 AudioJack2_SwitchT, J8 AudioJack2_SwitchT, J9 AudioJack2_SwitchT, Q1 MMBT3904, U1 MCP6002-xSN, U10 TL072, U11 TL072, U12 W25Q32JVSS, U13 TPS61040DBV, U14 W25Q32JVSS, U15 USBLC6-2SC6, U16 TL072, U17 LIS2DH12, U2 LM1117-3.3, U3 LM1117-3.3, U4 STM32L476VGTx, U5 TL072, U6 WM8758B, U7 TL072, U8 MCP6002-xSN, U9 MCP6002-xSN, Y1 Crystal_GND24

Commit message: add oss text to pcbs
Other:
- net class Default removed
- board text added: "this PCB is based on the opensource version of plinky available at https://github.com/plinkysynth/plinky_public this is not an official kit and is not officially supported"
