File: hw/testjig/testjig.kicad_sch (KiCad schematic)
At the start: 83 parts, among them J1 Conn_02x08_Odd_Even, J10 Conn_01x01, J11 Conn_01x01, J12 Conn_01x01, J13 Conn_01x01, J14 Conn_01x01, J15 Conn_01x01, J16 Conn_01x01, J17 Conn_01x01, J18 Conn_01x01, J19 Conn_01x01, J2 Conn_01x01, J20 Conn_01x04_Female, J21 Conn_01x01, J22 Conn_01x01, J23 Conn_01x01, J24 Conn_01x01, J25 Conn_01x01, J26 Conn_01x01, J27 Conn_01x01, J28 Conn_01x01, J29 Conn_01x01, J3 Conn_01x01, J30 Conn_01x01, J31 Conn_01x01, J32 Conn_01x01, J33 Conn_01x01, J34 Conn_01x01, J35 Conn_01x01, J36 Conn_01x01, J37 Conn_01x01, J38 Conn_01x01, J39 Conn_01x01, J4 Conn_01x01, J40 Conn_01x01, J41 Conn_01x01, J42 Conn_01x01, J43 Conn_02x08_Odd_Even, J44 USB_B_Micro, J45 Conn_02x07_Odd_Even, J46 Conn_01x04_Female, J47 Conn_01x06_Female, J48 Conn_01x02_Female, J49 Conn_01x01, J5 Conn_01x01, J50 Conn_01x01, J51 SJ1-3523N-cap, J52 Conn_01x04_Female, J6 Conn_01x01, J7 Conn_01x01, J8 Conn_01x01, J9 Conn_01x01, SW1 SW_Push_DPDT, SW2 SW_Push_DPDT, U1 CD74HC4067M

Commit message: Kicad files for Plinky v3, added testpoints and fixed Testjig
Parts:
- removed D6: LED_RABG, testjig:LED_RGB_1210_reverse, symbol Device:LED_RABG
- added D8: ASMB-MTB1-0A3A2, MSM_LED:C264508_Everlight, symbol LED:ASMB-MTB1-0A3A2
- added J1: PJ-320B, MyLibrary:LUOYANG-DISHANG_PJ-320B, symbol MICROMIDITRS-eagle-import:PJ-320B
- added JP1: SolderJumper_2_Bridged, Jumper:SolderJumper-2_P1.3mm_Bridged_RoundedPad1.0x1.5mm, symbol Jumper:SolderJumper_2_Bridged
Connections:
- net +3V3: now also D8.4 (A)
- net 5V: now also JP1.1 (A)
- net GND: now also J1.4 (SLEEVE)
- net VBUS: now also JP1.2 (B)
- net at R8.1: now also D8.1 (RK)
- net at R10.1: now also D8.3 (BK)
- net at R9.1: now also D8.2 (GK)
- net Test_HP_L: now reaches J21.1 (Pin_1), J51.2
- net Test_HP_L: now also J1.2 (TIP)
- net Test_HP_R: now reaches J50.1 (Pin_1), J51.3
- net Test_HP_R: now also J1.3 (RING)
