File: hw/plinkyblack/plinkyblack_hwmidi_jacks.kicad_sch (KiCad schematic)
At the start: 300 parts, among them J1 AudioJack2_SwitchT, J10 AudioJack2_SwitchT, J11 AudioJack2_SwitchT, J12 Conn_02x08_Odd_Even, J13 Conn_02x08_Odd_Even, J14 AudioJack2_SwitchT, J15 AudioJack2_SwitchT, J16 AudioJack2_SwitchT, J17 AudioJack2_SwitchT, J2 AudioJack2_SwitchT, J20 oled0.91, J22 AudioJack2_SwitchT, J23 AudioJack2_SwitchT, J25 Conn_01x16_Female, J28 PJ313, J29 PJ313, J3 AudioJack2_SwitchT, J30 PJ313, J31 PJ313, J32 PJ313, J33 PJ313, J4 AudioJack2_SwitchT, J5 SWD header, J6 AudioJack2_SwitchT, J7 AudioJack2_SwitchT, J8 AudioJack2_SwitchT, J9 AudioJack2_SwitchT, Q1 MMBT3904, U1 HCPL-0631-500E, U1 MCP6002-xSN, U10 TL072, U11 TL072, U12 W25Q32JVSS, U13 TPS61040DBV, U14 W25Q32JVSS, U15 WE-TVS-824001, U16 TL072, U17 LIS2DH12, U18 TL072, U19 TYPE-C-31-M-14, U2 LM1117-3.3, U20 TYPE-C-31-M-14, U22 PI3USB102EZLE, U23 WE-TVS-824001, U3 LM1117-3.3, U4 STM32L476VGT6, U5 TL072, U6 WM8758B, U7 TL072, U8 MCP6002-xSN, U9 MCP6002-xSN, Y1 Crystal_GND24

Commit message: Name mini jack connectors in schematic
Parts:
- renumbered C2 to C81, R3 to R107, R4 to R108, R5 to R109, R1 to R110, R6 to R111, R7 to R112, R2 to R113, U1 to U21
Other:
- note added: "CLOCK"
- note added: "EURO AUDIO IN"
- note added: "EURO CLOCK IN"
- note added: "EURO GATE IN"
- note added: "EURO OUT L"
- note added: "EURO OUT R"
- note added: "EURO PITCH IN"
- note added: "GATE"
- note added: "LFO A IN"
- note added: "LFO B IN"
- note added: "LFO X IN"
- note added: "LFO Y IN"
- note added: "LINE IN BOTTOM"
- note added: "LINE IN TOP"
- note added: "PHONES OUT BOTTOM"
- note added: "PHONES OUT TOP"
- note added: "PITCH HI"
- note added: "PITCH LO"
- note added: "PRESSURE"
- note added: "TRIGGER"
- note removed: "pitch"
- moved on the sheet: C41, U9C
